Commit message: rm redundant ns

File: trina2_description/base/urdf/freight.urdf.xacro (robot description, xacro)
@@ -117,5 +117,4 @@
     <axis xyz="0 0 0" />
   </joint>
-  <!-- TEMPORARY FIX -->
   <link name="laser_link">
     <inertial>
@@ -146,16 +145,4 @@
     <axis xyz="0 0 0" />
   </joint>
-  <link name="base_camera_link" />
-  <joint name="base_camera_joint" type="fixed">
-    <origin rpy="0 -0.17453292519943 0" xyz="0.2645 0 0.198" />
-    <parent link="chassis_link" />
-    <child link="base_camera_link" />
-  </joint>
-  <link name="base_camera_optical_frame" />
-  <joint name="base_camera_optical_joint" type="fixed">
-    <origin rpy="1.5707963267966 0 1.5707963267966" xyz="0 0 0" />
-    <parent link="base_camera_link" />
-    <child link="base_camera_optical_frame" />
-  </joint>
   <transmission name="r_wheel_trans">
     <type>transmission_interface/SimpleTransmission</type>

File: trina2_description/base/urdf/freight_macro.xacro (robot description, xacro)
@@ -1,5 +1,5 @@
 <?xml version="1.0"?>
 <robot name="freight" xmlns:xacro="http://www.ros.org/wiki/xacro">
-  <xacro:macro name="load_base" params="ns">
+  <xacro:macro name="load_base">
       <!-- <xacro:include filename="$(find fetch_description)/robots/freight.urdf.xacro" /> -->
       <xacro:include filename="$(find trina2_description)/base/urdf/freight.urdf.xacro" />

File: trina2_description/base/urdf/torso.urdf.xacro (robot description, xacro)
@@ -1,5 +1,5 @@
 <?xml version="1.0"?>
 <robot name="robot_torso" xmlns:xacro="http://www.ros.org/wiki/xacro">
-    <xacro:macro name="load_torso" params="ns">
+    <xacro:macro name="load_torso">
         <xacro:property name="mass" value="5.0" />
         <xacro:property name="width" value="0.15" />
@@ -36,5 +36,5 @@
             <axis xyz="0 0 1"/>
         </joint>
-        <link name="right_shoulder">
+        <link name="right_shoulder_link">
             <collision>
             <origin xyz="0 0 0" rpy="0 0 0"/>
@@ -57,11 +57,11 @@
             </inertial>
         </link>
-        <joint name="right_shoulder_to_torso" type="fixed">
-            <child link="right_shoulder" />
+        <joint name="right_shoulder_to_torso_joint" type="fixed">
+            <child link="right_shoulder_link" />
             <parent link="torso" />
             <origin xyz="0 0 0.7" rpy="1.57 0 0" />
             <axis xyz="0 0 1"/>
         </joint>
-        <link name="left_shoulder">
+        <link name="left_shoulder_link">
             <collision>
             <origin xyz="0 0 0" rpy="0 0 0"/>
@@ -84,6 +84,6 @@
             </inertial>
         </link>
-        <joint name="left_shoulder_to_torso" type="fixed">
-            <child link="left_shoulder" />
+        <joint name="left_shoulder_to_torso_joint" type="fixed">
+            <child link="left_shoulder_link" />
             <parent link="torso" />
             <origin xyz="0 0 0.7" rpy="-1.57 0 0" />

File: trina2_description/camera/urdf/arm_camera.urdf.xacro (robot description, xacro)
@@ -1,5 +1,5 @@
 <?xml version="1.0"?>
 <robot name="main_camera" xmlns:xacro="http://www.ros.org/wiki/xacro">
-    <xacro:macro name="load_arm_camera" params="ns prefix arm_camera_base
+    <xacro:macro name="load_arm_camera" params="prefix arm_camera_base
                                                 fov:=69.4 width:=1920 height:=1080
                                                 update_rate:=60 wide_flag:=true">
@@ -32,5 +32,5 @@
         </joint>
         <xacro:include filename="$(find trina2_description)/camera/urdf/_d435.urdf.xacro"/>
-        <xacro:sensor_d435 name="${prefix}cam" topics_ns="${ns}" parent="${prefix}camera_support"
+        <xacro:sensor_d435 name="${prefix}cam" parent="${prefix}camera_support"
                            fov="${fov}" width="${width}" height="${height}"
                            update_rate="${update_rate}" wide_flag="${wide_flag}">

File: trina2_description/camera/urdf/main_camera_support.urdf.xacro (robot description, xacro)
@@ -1,5 +1,5 @@
 <?xml version="1.0"?>
 <robot name="main_camera" xmlns:xacro="http://www.ros.org/wiki/xacro">
-    <xacro:macro name="load_main_camera" params="ns prefix main_camera_base
+    <xacro:macro name="load_main_camera" params="prefix main_camera_base
                                                  fov:=69.4 width:=1920 height:=1080
                                                  update_rate:=60 wide_flag:=true">
@@ -119,5 +119,5 @@
         </transmission>
         <xacro:include filename="$(find trina2_description)/camera/urdf/_d435.urdf.xacro"/>
-        <xacro:sensor_d435 name="${prefix}cam" topics_ns="${ns}" parent="${prefix}camera_pitch_link"
+        <xacro:sensor_d435 name="${prefix}cam" parent="${prefix}camera_pitch_link"
                            fov="${fov}" width="${width}" height="${height}"
                            update_rate="${update_rate}"  wide_flag="${wide_flag}">

File: trina2_description/robots/urdf/trina2.xacro (robot description, xacro)
@@ -5,7 +5,6 @@
     <xacro:arg name="dof" default="7" />
     <xacro:arg name="vision" default="true" />
-    <xacro:arg name="gripper" default="false" />
+    <xacro:arg name="gripper" default="robotiq_2f_85" />
     <xacro:arg name="sim" default="true" />
-    <xacro:arg name="ns" default="trina2" />
     <xacro:arg name="right_prefix" default="right_arm_" />
     <xacro:arg name="left_prefix" default="left_arm_" />
@@ -17,23 +16,23 @@
     <xacro:include filename="$(find trina2_description)/camera/urdf/arm_camera.urdf.xacro" />
     <!-- Load the base -->
-    <xacro:load_base ns="$(arg ns)"/>
+    <xacro:load_base/>
     <!-- Load torso -->
-    <xacro:load_torso ns="$(arg ns)"/>
+    <xacro:load_torso/>
     <!-- Load the right arm -->
     <xacro:load_robot arm="$(arg arm)" gripper="$(arg gripper)" dof="$(arg dof)"
                     vision="$(arg vision)" sim="$(arg sim)"
-                    prefix="$(arg right_prefix)" parent="right_shoulder"/>
+                    prefix="$(arg right_prefix)" parent="right_shoulder_link"/>
     <!-- Load arm camera -->
-    <xacro:load_arm_camera ns="$(arg ns)" prefix="$(arg right_prefix)" arm_camera_base="$(arg right_prefix)camera_link"
+    <xacro:load_arm_camera prefix="$(arg right_prefix)" arm_camera_base="$(arg right_prefix)camera_link"
                            width="858" height="720" update_rate="30" wide_flag="true"/>
     <!-- Load the left arm -->
     <xacro:load_robot arm="$(arg arm)" gripper="$(arg gripper)" dof="$(arg dof)"
                     vision="$(arg vision)" sim="$(arg sim)"
-                    prefix="$(arg left_prefix)" parent="left_shoulder"/>
+                    prefix="$(arg left_prefix)" parent="left_shoulder_link"/>
     <!-- Load arm camera -->
-    <xacro:load_arm_camera ns="$(arg ns)" prefix="$(arg left_prefix)" arm_camera_base="$(arg left_prefix)camera_link"
+    <xacro:load_arm_camera prefix="$(arg left_prefix)" arm_camera_base="$(arg left_prefix)camera_link"
                            width="858" height="720" update_rate="30" wide_flag="true"/>
     <!-- Load main camera -->
-    <xacro:load_main_camera ns="$(arg ns)" prefix="main_" main_camera_base="torso"
+    <xacro:load_main_camera prefix="main_" main_camera_base="torso"
                             width="858" height="720" update_rate="30" wide_flag="true"/>
     <!-- Load gazebo control pulgin ONLY ONCE -->
