Commit message: improve camera performance

File: trina2_description/arms/urdf/kortex_robot.xacro (robot description, xacro)
@@ -1,5 +1,5 @@
 <?xml version="1.0"?>
 <robot xmlns:xacro="http://ros.org/wiki/xacro">
-    <xacro:macro name="load_robot" params="arm gripper dof vision sim prefix">
+    <xacro:macro name="load_robot" params="arm gripper dof vision sim prefix parent">
         <!-- Files to include -->
         <xacro:include filename="$(find kortex_description)/arms/${arm}/${dof}dof/urdf/${arm}_macro.xacro" />
@@ -16,13 +16,12 @@
         </xacro:if>
         <!-- Run the macros -->
-        <!-- For gazebo
+        <!-- For gazebo -->
         <xacro:if value="${sim}">
-            <link name="world" />
-            <joint name="world_to_root" type="fixed">
+            <joint name="${parent}_to_${prefix}root" type="fixed">
                 <child link="${prefix}base_link" />
-                <parent link="world" />
+                <parent link="${parent}" />
                 <origin xyz="0 0 0" rpy="0 0 0" />
             </joint>
-        </xacro:if>-->
+        </xacro:if>
         <!-- Load the arm -->
         <xacro:load_arm parent="" dof="${dof}" vision="${vision}" prefix="${prefix}">

File: trina2_description/base/urdf/torso.urdf.xacro (robot description, xacro)
@@ -4,17 +4,17 @@
         <xacro:property name="mass" value="5.0" />
         <xacro:property name="width" value="0.15" />
-        <xacro:property name="height1" value="0.8" />
+        <xacro:property name="height" value="0.8" />
         <xacro:property name="axel_offset" value="-0.25" />
         <link name="torso">
             <collision>
-                <origin xyz="0 0 ${height1/2}" rpy="0 0 0"/>
+                <origin xyz="0 0 ${height/2}" rpy="0 0 0"/>
                 <geometry>
-                    <box size="${width} ${width} ${height1}"/>
+                    <box size="${width} ${width} ${height}"/>
                 </geometry>
             </collision>
             <visual>
-                <origin xyz="0 0 ${height1/2}" rpy="0 0 0"/>
+                <origin xyz="0 0 ${height/2}" rpy="0 0 0"/>
                 <geometry>
-                    <box size="${width} ${width} ${height1}"/>
+                    <box size="${width} ${width} ${height}"/>
                 </geometry>
                 <material name="">
@@ -23,8 +23,8 @@
             </visual>
             <inertial>
-                <origin xyz="0 0 ${height1/2}" rpy="0 0 0"/>
+                <origin xyz="0 0 ${height/2}" rpy="0 0 0"/>
                 <mass value="${mass}"/>
-                <inertia ixx="${mass / 12.0 * (width*width + height1*height1)}" ixy="0.0" ixz="0.0"
-                        iyy="${mass / 12.0 * (height1*height1 + width*width)}" iyz="0.0"
+                <inertia ixx="${mass / 12.0 * (width*width + height*height)}" ixy="0.0" ixz="0.0"
+                        iyy="${mass / 12.0 * (height*height + width*width)}" iyz="0.0"
                         izz="${mass / 12.0 * (width*width + width*width)}"/>
             </inertial>
@@ -36,4 +36,58 @@
             <axis xyz="0 0 1"/>
         </joint>
+        <link name="right_shoulder">
+            <collision>
+            <origin xyz="0 0 0" rpy="0 0 0"/>
+            <geometry>
+                <box size="0.001 0.001 0.001"/>
+            </geometry>
+            </collision>
+            <visual>
+            <origin xyz="0 0 0" rpy="0 0 0"/>
+            <geometry>
+                <box size="0.001 0.001 0.001"/>
+            </geometry>
+            </visual>
+            <inertial>
+            <origin xyz="0 0 0" rpy="0 0 0"/>
+            <mass value="0.0"/>
+            <inertia ixx="0.01" ixy="0.01" ixz="0.01"
+                     iyy="0.01" iyz="0.01"
+                     izz="0.01"/>
+            </inertial>
+        </link>
+        <joint name="right_shoulder_to_torso" type="fixed">
+            <child link="right_shoulder" />
+            <parent link="torso" />
+            <origin xyz="0 0 0.7" rpy="1.57 0 0" />
+            <axis xyz="0 0 1"/>
+        </joint>
+        <link name="left_shoulder">
+            <collision>
+            <origin xyz="0 0 0" rpy="0 0 0"/>
+            <geometry>
+                <box size="0.001 0.001 0.001"/>
+            </geometry>
+            </collision>
+            <visual>
+            <origin xyz="0 0 0" rpy="0 0 0"/>
+            <geometry>
+                <box size="0.001 0.001 0.001"/>
+            </geometry>
+            </visual>
+            <inertial>
+            <origin xyz="0 0 0" rpy="0 0 0"/>
+            <mass value="0.0"/>
+            <inertia ixx="0.01" ixy="0.01" ixz="0.01"
+                     iyy="0.01" iyz="0.01"
+                     izz="0.01"/>
+            </inertial>
+        </link>
+        <joint name="left_shoulder_to_torso" type="fixed">
+            <child link="left_shoulder" />
+            <parent link="torso" />
+            <origin xyz="0 0 0.7" rpy="-1.57 0 0" />
+            <axis xyz="0 0 1"/>
+        </joint>
     </xacro:macro>
 </robot>

File: trina2_description/camera/urdf/_d435.gazebo.xacro (robot description, xacro)
@@ -1,143 +1,56 @@
 <?xml version="1.0"?>
 <!--
-License: Apache 2.0. See LICENSE file in root directory.
-Copyright(c) 2017 PAL Robotics, S.L. All Rights Reserved
 This is the Gazebo URDF model for the Intel RealSense D435 camera
+using libgazebo_ros_openni_kinect plugin
 -->
 <robot xmlns:xacro="http://ros.org/wiki/xacro">
-  <xacro:macro name="gazebo_d435" params="camera_name reference_link topics_ns
-                                          depth_optical_frame color_optical_frame
-                                          infrared1_optical_frame infrared2_optical_frame
-                                          color_fov:=69.4 color_w:=1920 color_h:=1080
-                                          depth_fov:=85.2 depth_w:=1280 depth_h:=720
-                                          update_rate:=60" >
+  <xacro:macro name="gazebo_d435" params="camera_name reference_link
+                                          topics_ns color_optical_frame
+                                          fov:=69.4 width:=1920 height:=1080
+                                          update_rate:=30" >
     <!-- Load parameters to model's main link-->
     <xacro:property name="deg_to_rad" value="0.01745329251994329577" />
     <gazebo reference="${reference_link}">
-      <self_collide>0</self_collide>
-      <enable_wind>0</enable_wind>
-      <kinematic>0</kinematic>
-      <!-- <gravity>1</gravity> -->
-      <!--<mu>1</mu>-->
-      <mu2>1</mu2>
-      <fdir1>0 0 0</fdir1>
-      <!--<slip1>0</slip1>
-      <slip2>0</slip2>-->
-      <kp>1e+13</kp>
-      <kd>1</kd>
-      <!--<max_vel>0.01</max_vel>
-      <min_depth>0</min_depth>-->
-      <sensor name="${camera_name}color" type="camera">
-        <camera name="${camera_name}">
-          <horizontal_fov>${color_fov*deg_to_rad}</horizontal_fov>
+      <sensor type="depth" name="${camera_name}">
+        <always_on>1</always_on>
+        <update_rate>${update_rate}</update_rate>
+        <visualize>false</visualize>
+        <camera>
+          <horizontal_fov>${fov*deg_to_rad}</horizontal_fov>
           <image>
-            <width>${color_w}</width>
-            <height>${color_h}</height>
-            <format>RGB_INT8</format>
+            <width>${width}</width>
+            <height>${height}</height>
+            <format>R8G8B8</format>
           </image>
           <clip>
             <near>0.1</near>
-            <far>100</far>
+            <far>20</far>
           </clip>
-          <noise>
-            <type>gaussian</type>
-            <mean>0.0</mean>
-            <stddev>0.007</stddev>
-          </noise>
         </camera>
-        <always_on>1</always_on>
-        <update_rate>${update_rate}</update_rate>
-        <visualize>0</visualize>
+        <plugin name="${camera_name}_controller" filename="libgazebo_ros_openni_kinect.so">
+          <baseline>0.2</baseline>
+          <alwaysOn>true</alwaysOn>
+          <updateRate>0.0</updateRate>
+          <cameraName>${camera_name}</cameraName>
+          <frameName>${color_optical_frame}</frameName>
+          <imageTopicName>color/image_raw</imageTopicName>
+          <depthImageTopicName>depth/image_raw</depthImageTopicName>
+          <pointCloudTopicName>depth/points</pointCloudTopicName>
+          <cameraInfoTopicName>color/camera_info</cameraInfoTopicName>
+          <depthImageCameraInfoTopicName>depth/camera_info</depthImageCameraInfoTopicName>
+          <pointCloudCutoff>0.5</pointCloudCutoff>
+          <pointCloudCutoffMax>3.0</pointCloudCutoffMax>
+          <distortionK1>0</distortionK1>
+          <distortionK2>0</distortionK2>
+          <distortionK3>0</distortionK3>
+          <distortionT1>0</distortionT1>
+          <distortionT2>0</distortionT2>
+          <CxPrime>0</CxPrime>
+          <Cx>0</Cx>
+          <Cy>0</Cy>
+          <focalLength>0</focalLength>
+          <hackBaseline>0</hackBaseline>
+        </plugin>
       </sensor>
-      <sensor name="${camera_name}ired1" type="camera">
-        <camera name="${camera_name}">
-          <horizontal_fov>${depth_fov*deg_to_rad}</horizontal_fov>
-          <image>
-            <width>${depth_w}</width>
-            <height>${depth_h}</height>
-            <format>L_INT8</format>
-          </image>
-          <clip>
-            <near>0.1</near>
-            <far>100</far>
-          </clip>
-          <noise>
-            <type>gaussian</type>
-            <mean>0.0</mean>
-            <stddev>0.05</stddev>
-          </noise>
-        </camera>
-        <always_on>0</always_on>
-        <update_rate>${update_rate}</update_rate>
-        <visualize>0</visualize>
-      </sensor>
-      <sensor name="${camera_name}ired2" type="camera">
-        <camera name="${camera_name}">
-          <horizontal_fov>${depth_fov*deg_to_rad}</horizontal_fov>
-          <image>
-            <width>${depth_w}</width>
-            <height>${depth_h}</height>
-            <format>L_INT8</format>
-          </image>
-          <clip>
-            <near>0.1</near>
-            <far>100</far>
-          </clip>
-          <noise>
-            <type>gaussian</type>
-            <mean>0.0</mean>
-            <stddev>0.05</stddev>
-          </noise>
-        </camera>
-        <always_on>0</always_on>
-        <update_rate>${update_rate}</update_rate>
-        <visualize>0</visualize>
-      </sensor>
-      <sensor name="${camera_name}depth" type="depth">
-        <camera name="${camera_name}">
-          <horizontal_fov>${depth_fov*deg_to_rad}</horizontal_fov>
-          <image>
-            <width>${depth_w}</width>
-            <height>${depth_h}</height>
-          </image>
-          <clip>
-            <near>0.1</near>
-            <far>100</far>
-          </clip>
-          <noise>
-            <type>gaussian</type>
-            <mean>0.0</mean>
-            <stddev>0.100</stddev>
-          </noise>
-        </camera>
-        <always_on>0</always_on>
-        <update_rate>${update_rate}</update_rate>
-        <visualize>0</visualize>
-      </sensor>
-    </gazebo>
-    <gazebo>
-      <plugin name="${topics_ns}" filename="librealsense_gazebo_plugin.so">
-        <prefix>${camera_name}</prefix>
-      	<depthUpdateRate>${update_rate}</depthUpdateRate>
-      	<colorUpdateRate>${update_rate}</colorUpdateRate>
-      	<infraredUpdateRate>${update_rate}</infraredUpdateRate>
-      	<depthTopicName>depth/image_raw</depthTopicName>
-      	<depthCameraInfoTopicName>depth/camera_info</depthCameraInfoTopicName>
-      	<colorTopicName>color/image_raw</colorTopicName>
-      	<colorCameraInfoTopicName>color/camera_info</colorCameraInfoTopicName>
-      	<infrared1TopicName>infra1/image_raw</infrared1TopicName>
-      	<infrared1CameraInfoTopicName>infra1/camera_info</infrared1CameraInfoTopicName>
-      	<infrared2TopicName>infra2/image_raw</infrared2TopicName>
-      	<infrared2CameraInfoTopicName>infra2/camera_info</infrared2CameraInfoTopicName>
-      	<colorOpticalframeName>${color_optical_frame}</colorOpticalframeName>
-      	<depthOpticalframeName>${depth_optical_frame}</depthOpticalframeName>
-      	<infrared1OpticalframeName>${infrared1_optical_frame}</infrared1OpticalframeName>
-      	<infrared2OpticalframeName>${infrared2_optical_frame}</infrared2OpticalframeName>
-      	<rangeMinDepth>0.2</rangeMinDepth>
-      	<rangeMaxDepth>10.0</rangeMaxDepth>
-      	<pointCloud>false</pointCloud>
-      	<pointCloudTopicName>depth/points</pointCloudTopicName>
-      	<pointCloudCutoff>0.5</pointCloudCutoff>
-      </plugin>
     </gazebo>
   </xacro:macro>

File: trina2_description/camera/urdf/_d435.urdf.xacro (robot description, xacro)
@@ -3,5 +3,5 @@
 License: Apache 2.0. See LICENSE file in root directory.
 Copyright(c) 2017 Intel Corporation. All Rights Reserved
-This is the URDF model for the Intel RealSense 430 camera, in it's
+This is the URDF model for the Intel RealSense 435 camera, in it's
 aluminum peripherial evaluation case.
 -->
@@ -10,6 +10,5 @@
   <xacro:include filename="$(find trina2_description)/camera/urdf/_d435.gazebo.xacro"/>
   <xacro:macro name="sensor_d435" params="name:=camera topics_ns:=camera parent
-                                          color_fov:=69.4 color_w:=1920 color_h:=1080
-                                          depth_fov:=85.2 depth_w:=1280 depth_h:=720
+                                          fov:=69.4 width:=1920 height:=1080
                                           update_rate:=60 wide_flag:=false *origin">
     <xacro:property name="M_PI" value="3.1415926535897931" />
@@ -126,20 +125,14 @@
     <!-- Normal camera -->
     <xacro:gazebo_d435 camera_name="${name}" reference_link="${name}_link"
-                      topics_ns="${topics_ns}" depth_optical_frame="${name}_depth_optical_frame"
+                      topics_ns="${topics_ns}"
                       color_optical_frame="${name}_color_optical_frame"
-                      infrared1_optical_frame="${name}_left_ir_optical_frame"
-                      infrared2_optical_frame="${name}_right_ir_optical_frame"
-                      color_fov="${color_fov}" color_w="${color_w}" color_h="${color_h}"
-                      depth_fov="${depth_fov}" depth_w="${depth_w}" depth_h="${depth_h}"
+                      fov="${fov}" width="${width}" height="${height}"
                       update_rate="${update_rate}"/>
     <!-- Wide camera -->
     <xacro:if value="${wide_flag}">
     <xacro:gazebo_d435 camera_name="${name}_wide" reference_link="${name}_link"
-                      topics_ns="${topics_ns}_wide" depth_optical_frame="${name}_depth_optical_frame"
+                      topics_ns="${topics_ns}_wide"
                       color_optical_frame="${name}_color_optical_frame"
-                      infrared1_optical_frame="${name}_left_ir_optical_frame"
-                      infrared2_optical_frame="${name}_right_ir_optical_frame"
-                      color_fov="114" color_w="${1.3125*color_w}" color_h="${color_h}"
-                      depth_fov="${depth_fov}" depth_w="${depth_w}" depth_h="${depth_h}"
+                      fov="114" width="${1.3125*width}" height="${height}"
                       update_rate="${update_rate}"/>
     </xacro:if>

File: trina2_description/camera/urdf/arm_camera.urdf.xacro (robot description, xacro)
@@ -2,6 +2,5 @@
 <robot name="main_camera" xmlns:xacro="http://www.ros.org/wiki/xacro">
     <xacro:macro name="load_arm_camera" params="ns prefix arm_camera_base
-                                                color_fov:=69.4 color_w:=1920 color_h:=1080
-                                                depth_fov:=85.2 depth_w:=1280 depth_h:=720
+                                                fov:=69.4 width:=1920 height:=1080
                                                 update_rate:=60 wide_flag:=true">
         <link name="${prefix}camera_support">
@@ -33,7 +32,6 @@
         </joint>
         <xacro:include filename="$(find trina2_description)/camera/urdf/_d435.urdf.xacro"/>
-        <xacro:sensor_d435 name="${prefix}cam" topics_ns="${prefix}cam" parent="${prefix}camera_support"
-                           color_fov="${color_fov}" color_w="${color_w}" color_h="${color_h}"
-                           depth_fov="${depth_fov}" depth_w="${depth_w}" depth_h="${depth_h}"
+        <xacro:sensor_d435 name="${prefix}cam" topics_ns="${ns}" parent="${prefix}camera_support"
+                           fov="${fov}" width="${width}" height="${height}"
                            update_rate="${update_rate}" wide_flag="${wide_flag}">
             <origin xyz="0.0 0.0 0.0" rpy="0 0 0" />

File: trina2_description/camera/urdf/main_camera_support.urdf.xacro (robot description, xacro)
@@ -2,22 +2,21 @@
 <robot name="main_camera" xmlns:xacro="http://www.ros.org/wiki/xacro">
     <xacro:macro name="load_main_camera" params="ns prefix main_camera_base
-                                                 color_fov:=69.4 color_w:=1920 color_h:=1080
-                                                 depth_fov:=85.2 depth_w:=1280 depth_h:=720
+                                                 fov:=69.4 width:=1920 height:=1080
                                                  update_rate:=60 wide_flag:=true">
         <xacro:property name="mass" value="0.2" />
-        <xacro:property name="width" value="0.04" />
-        <xacro:property name="height1" value="0.02" />
+        <xacro:property name="width_support" value="0.04" />
+        <xacro:property name="height_support" value="0.02" />
         <xacro:property name="axel_offset" value="-0.25" />
         <link name="${prefix}camera_support">
             <collision>
-            <origin xyz="0 0 ${height1/2}" rpy="0 0 0"/>
+            <origin xyz="0 0 ${height_support/2}" rpy="0 0 0"/>
             <geometry>
-                <box size="${width} ${width} ${height1}"/>
+                <box size="${width_support} ${width_support} ${height_support}"/>
             </geometry>
             </collision>
             <visual>
-            <origin xyz="0 0 ${height1/2}" rpy="0 0 0"/>
+            <origin xyz="0 0 ${height_support/2}" rpy="0 0 0"/>
             <geometry>
-                <box size="${width} ${width} ${height1}"/>
+                <box size="${width_support} ${width_support} ${height_support}"/>
             </geometry>
             <material name="">
@@ -26,9 +25,9 @@
             </visual>
             <inertial>
-            <origin xyz="0 0 ${height1/2}" rpy="0 0 0"/>
+            <origin xyz="0 0 ${height_support/2}" rpy="0 0 0"/>
             <mass value="${mass}"/>
-            <inertia ixx="${mass / 12.0 * (width*width + height1*height1)}" ixy="0.0" ixz="0.0"
-                    iyy="${mass / 12.0 * (height1*height1 + width*width)}" iyz="0.0"
-                    izz="${mass / 12.0 * (width*width + width*width)}"/>
+            <inertia ixx="${mass / 12.0 * (width_support*width_support + height_support*height_support)}" ixy="0.0" ixz="0.0"
+                    iyy="${mass / 12.0 * (height_support*height_support + width_support*width_support)}" iyz="0.0"
+                    izz="${mass / 12.0 * (width_support*width_support + width_support*width_support)}"/>
             </inertial>
         </link>
@@ -36,5 +35,5 @@
             <parent link="${main_camera_base}"/>
             <child link="${prefix}camera_support"/>
-            <origin xyz="${0.075-width/2} 0 0.8" rpy="0 0 0"/>
+            <origin xyz="${0.075-width_support/2} 0 0.8" rpy="0 0 0"/>
             <axis xyz="0 0 1"/>
         </joint>
@@ -66,5 +65,5 @@
             <parent link="${prefix}camera_support"/>
             <child link="${prefix}camera_yaw_link"/>
-            <origin xyz="0 0 ${height1}" rpy="0 0 0"/>
+            <origin xyz="0 0 ${height_support}" rpy="0 0 0"/>
             <axis xyz="0 0 1"/>
             <limit lower="-1.047" upper="1.047" effort="20" velocity="1.0" />
@@ -120,7 +119,6 @@
         </transmission>
         <xacro:include filename="$(find trina2_description)/camera/urdf/_d435.urdf.xacro"/>
-        <xacro:sensor_d435 name="${prefix}cam" topics_ns="${prefix}cam" parent="${prefix}camera_pitch_link"
-                           color_fov="${color_fov}" color_w="${color_w}" color_h="${color_h}"
-                           depth_fov="${depth_fov}" depth_w="${depth_w}" depth_h="${depth_h}"
+        <xacro:sensor_d435 name="${prefix}cam" topics_ns="${ns}" parent="${prefix}camera_pitch_link"
+                           fov="${fov}" width="${width}" height="${height}"
                            update_rate="${update_rate}"  wide_flag="${wide_flag}">
             <origin xyz="0.02 0.0 0.0" rpy="-1.57 0 0" />
