Commit message: improve camera performance

File: trina2_description/robots/urdf/trina2.xacro (robot description, xacro)
@@ -5,5 +5,5 @@
     <xacro:arg name="dof" default="7" />
     <xacro:arg name="vision" default="true" />
-    <xacro:arg name="gripper" default="robotiq_2f_85" />
+    <xacro:arg name="gripper" default="false" />
     <xacro:arg name="sim" default="true" />
     <xacro:arg name="ns" default="trina2" />
@@ -11,40 +11,30 @@
     <xacro:arg name="left_prefix" default="left_arm_" />
     <!-- Include files -->
-    <xacro:include filename="$(find trina2_description)/arms/urdf/kortex_robot.xacro" />
     <xacro:include filename="$(find trina2_description)/base/urdf/freight_macro.xacro" />
     <xacro:include filename="$(find trina2_description)/base/urdf/torso.urdf.xacro" />
+    <xacro:include filename="$(find trina2_description)/arms/urdf/kortex_robot.xacro" />
     <xacro:include filename="$(find trina2_description)/camera/urdf/main_camera_support.urdf.xacro" />
     <xacro:include filename="$(find trina2_description)/camera/urdf/arm_camera.urdf.xacro" />
-    <!-- Load the right arm -->
-    <joint name="right_arm_to_torso" type="fixed">
-        <child link="$(arg right_prefix)base_link" />
-        <parent link="torso" />
-        <origin xyz="0 0 0.7" rpy="1.57 0 0" />
-        <axis xyz="0 0 1"/>
-    </joint>
-    <xacro:load_robot arm="$(arg arm)" gripper="$(arg gripper)" dof="$(arg dof)"
-                    vision="$(arg vision)" sim="$(arg sim)" prefix="$(arg right_prefix)"/>
-    <!-- Load arm camera -->
-    <xacro:load_arm_camera ns="$(arg ns)" prefix="$(arg right_prefix)" arm_camera_base="$(arg right_prefix)camera_link"
-                           color_w="1280" color_h="720" depth_w="858" depth_h="480" update_rate="30" wide_flag="true"/>
-    <!-- Load the left arm -->
-    <joint name="left_arm_to_torso" type="fixed">
-        <child link="$(arg left_prefix)base_link" />
-        <parent link="torso" />
-        <origin xyz="0 0 0.7" rpy="-1.57 0 0" />
-        <axis xyz="0 0 1"/>
-    </joint>
-    <xacro:load_robot arm="$(arg arm)" gripper="$(arg gripper)" dof="$(arg dof)"
-                    vision="$(arg vision)" sim="$(arg sim)" prefix="$(arg left_prefix)"/>
-    <!-- Load arm camera -->
-    <xacro:load_arm_camera ns="$(arg ns)" prefix="$(arg left_prefix)" arm_camera_base="$(arg left_prefix)camera_link"
-                           color_w="1280" color_h="720" depth_w="858" depth_h="480" update_rate="30" wide_flag="true"/>
-    <!-- Load main camera -->
-    <xacro:load_main_camera ns="$(arg ns)" prefix="main_" main_camera_base="torso"
-                            color_w="1280" color_h="720" depth_w="858" depth_h="480" update_rate="30" wide_flag="true"/>
     <!-- Load the base -->
     <xacro:load_base ns="$(arg ns)"/>
     <!-- Load torso -->
     <xacro:load_torso ns="$(arg ns)"/>
+    <!-- Load the right arm -->
+    <xacro:load_robot arm="$(arg arm)" gripper="$(arg gripper)" dof="$(arg dof)"
+                    vision="$(arg vision)" sim="$(arg sim)"
+                    prefix="$(arg right_prefix)" parent="right_shoulder"/>
+    <!-- Load arm camera -->
+    <xacro:load_arm_camera ns="$(arg ns)" prefix="$(arg right_prefix)" arm_camera_base="$(arg right_prefix)camera_link"
+                           width="858" height="720" update_rate="30" wide_flag="true"/>
+    <!-- Load the left arm -->
+    <xacro:load_robot arm="$(arg arm)" gripper="$(arg gripper)" dof="$(arg dof)"
+                    vision="$(arg vision)" sim="$(arg sim)"
+                    prefix="$(arg left_prefix)" parent="left_shoulder"/>
+    <!-- Load arm camera -->
+    <xacro:load_arm_camera ns="$(arg ns)" prefix="$(arg left_prefix)" arm_camera_base="$(arg left_prefix)camera_link"
+                           width="858" height="720" update_rate="30" wide_flag="true"/>
+    <!-- Load main camera -->
+    <xacro:load_main_camera ns="$(arg ns)" prefix="main_" main_camera_base="torso"
+                            width="858" height="720" update_rate="30" wide_flag="true"/>
     <!-- Load gazebo control pulgin ONLY ONCE -->
     <gazebo>

Commit message: add tf_prefix to urdf

File: trina2_description/arms/urdf/kortex_robot.xacro (robot description, xacro)
@@ -18,5 +18,5 @@
         <!-- For gazebo -->
         <xacro:if value="${sim}">
-            <joint name="${parent}_to_${prefix}root" type="fixed">
+            <joint name="${prefix}shoulder_to_arm_root" type="fixed">
                 <child link="${prefix}base_link" />
                 <parent link="${parent}" />

File: trina2_description/base/urdf/freight.urdf.xacro (robot description, xacro)
@@ -1,165 +1,179 @@
 <?xml version="1.0"?>
 <robot name="freight" xmlns:xacro="http://www.ros.org/wiki/xacro">
-  <link name="base_link"></link>
-  <joint name="base_link_joint" type="fixed">
-      <origin xyz="0 0 0" rpy="0 0 0" />
-      <parent link="base_link"/>
-      <child link="chassis_link" />
-  </joint>
-  <link name="chassis_link">
-    <inertial>
-      <origin rpy="0 0 0" xyz="-0.0036 0.0 0.0014" />
-      <mass value="70.1294" />
-      <inertia ixx="1.225" ixy="0.0099" ixz="0.0062" iyy="1.2853" iyz="-0.0034" izz="0.987" />
-    </inertial>
-    <visual>
-      <origin rpy="0 0 0" xyz="0 0 0" />
-      <geometry>
-        <mesh filename="package://trina2_description/base/meshes/base_link.dae" />
-      </geometry>
-      <material name="">
-        <color rgba="0.356 0.361 0.376 1" />
-      </material>
-    </visual>
-    <collision>
-      <origin rpy="0 0 0" xyz="0 0 0" />
-      <geometry>
-        <mesh filename="package://trina2_description/base/meshes/base_link_collision.STL" />
-      </geometry>
-    </collision>
-  </link>
-  <link name="r_wheel_link">
-    <inertial>
-      <origin rpy="0 0 0" xyz="0 0 0" />
-      <mass value="4.3542" />
-      <inertia ixx="0.0045" ixy="0" ixz="0" iyy="0.005" iyz="0" izz="0.0045" />
-    </inertial>
-    <visual>
-      <origin rpy="0 0 0" xyz="0 0 0" />
-      <geometry>
-        <mesh filename="package://trina2_description/base/meshes/r_wheel_link.STL" />
-      </geometry>
-      <material name="">
-        <color rgba="0.086 0.506 0.767 1" />
-      </material>
-    </visual>
-    <collision>
-      <origin rpy="0 0 0" xyz="0 0 0" />
-      <geometry>
-        <mesh filename="package://trina2_description/base/meshes/r_wheel_link_collision.STL" />
-      </geometry>
-    </collision>
-  </link>
-  <joint name="r_wheel_joint" type="continuous">
-    <!--origin rpy="-6.123E-17 0 0" xyz="0.0012914 -0.18738 0.055325" -->
-    <origin rpy="-6.123E-17 0 0" xyz="0.0012914 -0.18738 0.0602" />
-    <parent link="chassis_link" />
-    <child link="r_wheel_link" />
-    <axis xyz="0 1 0" />
-    <limit effort="8.85" velocity="34.8" />
-  </joint>
-  <link name="l_wheel_link">
-    <inertial>
-      <origin rpy="0 0 0" xyz="0 0 0" />
-      <mass value="4.3542" />
-      <inertia ixx="0.0045" ixy="0" ixz="0" iyy="0.005" iyz="0" izz="0.0045" />
-    </inertial>
-    <visual>
-      <origin rpy="0 0 0" xyz="0 0 0" />
-      <geometry>
-        <mesh filename="package://trina2_description/base/meshes/l_wheel_link.STL" />
-      </geometry>
-      <material name="">
-        <color rgba="0.086 0.506 0.767 1" />
-      </material>
-    </visual>
-    <collision>
-      <origin rpy="0 0 0" xyz="0 0 0" />
-      <geometry>
-        <mesh filename="package://trina2_description/base/meshes/l_wheel_link_collision.STL" />
-      </geometry>
-    </collision>
-  </link>
-  <joint name="l_wheel_joint" type="continuous">
-    <!-- origin rpy="-6.123E-17 0 0" xyz="0.0012914 0.18738 0.055325" -->
-    <origin rpy="-6.123E-17 0 0" xyz="0.0012914 0.18738 0.0602" />
-    <parent link="chassis_link" />
-    <child link="l_wheel_link" />
-    <axis xyz="0 1 0" />
-    <limit effort="8.85" velocity="34.8" />
-  </joint>
-  <link name="estop_link">
-    <inertial>
-      <origin rpy="0 0 0" xyz="0.002434512737072 -0.00330608315239905 0.00665139196650039" />
-      <mass value="0.00196130439134723" />
-      <inertia ixx="3.02810026604417E-07" ixy="-1.5862023118056E-08" ixz="3.16561396557437E-08" iyy="2.93322917127605E-07" iyz="-4.28833522751273E-08" izz="2.28513272627183E-07" />
-    </inertial>
-    <visual>
-      <origin rpy="0 0 0" xyz="0 0 0" />
-      <geometry>
-        <mesh filename="package://trina2_description/base/meshes/estop_link.STL" />
-      </geometry>
-      <material name="">
-        <color rgba="0.8 0 0 1" />
-      </material>
-    </visual>
-    <collision>
-      <origin rpy="0 0 0" xyz="0 0 0" />
-      <geometry>
-        <mesh filename="package://trina2_description/base/meshes/estop_link.STL" />
-      </geometry>
-    </collision>
-  </link>
-  <joint name="estop_joint" type="fixed">
-    <origin rpy="1.5708 0 0" xyz="-0.12465 0.23892 0.31127" />
-    <parent link="chassis_link" />
-    <child link="estop_link" />
-    <axis xyz="0 0 0" />
-  </joint>
-  <link name="laser_link">
-    <inertial>
-      <origin rpy="0 0 0" xyz="-0.0306228970175641 0.0007091682908278 0.0551974119471302" />
-      <mass value="0.00833634573995571" />
-      <inertia ixx="1.01866461240801E-06" ixy="-5.88447626567756E-08" ixz="7.83857244757914E-08" iyy="5.10039589974707E-07" iyz="-7.12664289617235E-09" izz="1.28270671527309E-06" />
-    </inertial>
-    <visual>
-      <origin rpy="0 0 0" xyz="0 0 0" />
-      <geometry>
-        <mesh filename="package://trina2_description/base/meshes/laser_link.STL" />
-      </geometry>
-      <material name="">
-        <color rgba="0.792156862745098 0.819607843137255 0.933333333333333 1" />
-      </material>
-    </visual>
-    <collision>
-      <origin rpy="0 0 0" xyz="0 0 0" />
-      <geometry>
-        <mesh filename="package://trina2_description/base/meshes/laser_link.STL" />
-      </geometry>
-    </collision>
-  </link>
-  <joint name="laser_joint" type="fixed">
-    <origin rpy="3.14159265359 0 0" xyz="0.235 0 0.2878" />
-    <parent link="chassis_link" />
-    <child link="laser_link" />
-    <axis xyz="0 0 0" />
-  </joint>
-  <transmission name="r_wheel_trans">
-    <type>transmission_interface/SimpleTransmission</type>
-    <joint name="r_wheel_joint">
-        <hardwareInterface>hardware_interface/VelocityJointInterface</hardwareInterface>
+  <xacro:macro name="load_base_urdf" params="prefix">
+    <link name="${prefix}base_link"></link>
+    <joint name="${prefix}base_link_joint" type="fixed">
+        <origin xyz="0 0 0" rpy="0 0 0" />
+        <parent link="${prefix}base_link"/>
+        <child link="${prefix}chassis_link" />
     </joint>
-    <actuator name="r_wheel_actuator">
-        <mechanicalReduction>1</mechanicalReduction>
-    </actuator>
-  </transmission>
-  <transmission name="l_wheel_trans">
-    <type>transmission_interface/SimpleTransmission</type>
-    <joint name="l_wheel_joint">
-        <hardwareInterface>hardware_interface/VelocityJointInterface</hardwareInterface>
+    <link name="${prefix}chassis_link">
+      <inertial>
+        <origin rpy="0 0 0" xyz="-0.0036 0.0 0.0014" />
+        <mass value="70.1294" />
+        <inertia ixx="1.225" ixy="0.0099" ixz="0.0062" iyy="1.2853" iyz="-0.0034" izz="0.987" />
+      </inertial>
+      <visual>
+        <origin rpy="0 0 0" xyz="0 0 0" />
+        <geometry>
+          <mesh filename="package://trina2_description/base/meshes/base_link.dae" />
+        </geometry>
+        <material name="">
+          <color rgba="0.356 0.361 0.376 1" />
+        </material>
+      </visual>
+      <collision>
+        <origin rpy="0 0 0" xyz="0 0 0" />
+        <geometry>
+          <mesh filename="package://trina2_description/base/meshes/base_link_collision.STL" />
+        </geometry>
+      </collision>
+    </link>
+    <link name="${prefix}r_wheel_link">
+      <inertial>
+        <origin rpy="0 0 0" xyz="0 0 0" />
+        <mass value="4.3542" />
+        <inertia ixx="0.0045" ixy="0" ixz="0" iyy="0.005" iyz="0" izz="0.0045" />
+      </inertial>
+      <visual>
+        <origin rpy="0 0 0" xyz="0 0 0" />
+        <geometry>
+          <mesh filename="package://trina2_description/base/meshes/r_wheel_link.STL" />
+        </geometry>
+        <material name="">
+          <color rgba="0.086 0.506 0.767 1" />
+        </material>
+      </visual>
+      <collision>
+        <origin rpy="0 0 0" xyz="0 0 0" />
+        <geometry>
+          <mesh filename="package://trina2_description/base/meshes/r_wheel_link_collision.STL" />
+        </geometry>
+      </collision>
+    </link>
+    <joint name="${prefix}r_wheel_joint" type="continuous">
+      <!--origin rpy="-6.123E-17 0 0" xyz="0.0012914 -0.18738 0.055325" -->
+      <origin rpy="-6.123E-17 0 0" xyz="0.0012914 -0.18738 0.0602" />
+      <parent link="${prefix}chassis_link" />
+      <child link="${prefix}r_wheel_link" />
+      <axis xyz="0 1 0" />
+      <limit effort="8.85" velocity="34.8" />
     </joint>
-    <actuator name="l_wheel_actuator">
-        <mechanicalReduction>1</mechanicalReduction>
-    </actuator>
-  </transmission>
+    <link name="${prefix}l_wheel_link">
+      <inertial>
+        <origin rpy="0 0 0" xyz="0 0 0" />
+        <mass value="4.3542" />
+        <inertia ixx="0.0045" ixy="0" ixz="0" iyy="0.005" iyz="0" izz="0.0045" />
+      </inertial>
+      <visual>
+        <origin rpy="0 0 0" xyz="0 0 0" />
+        <geometry>
+          <mesh filename="package://trina2_description/base/meshes/l_wheel_link.STL" />
+        </geometry>
+        <material name="">
+          <color rgba="0.086 0.506 0.767 1" />
+        </material>
+      </visual>
+      <collision>
+        <origin rpy="0 0 0" xyz="0 0 0" />
+        <geometry>
+          <mesh filename="package://trina2_description/base/meshes/l_wheel_link_collision.STL" />
+        </geometry>
+      </collision>
+    </link>
+    <joint name="${prefix}l_wheel_joint" type="continuous">
+      <!-- origin rpy="-6.123E-17 0 0" xyz="0.0012914 0.18738 0.055325" -->
+      <origin rpy="-6.123E-17 0 0" xyz="0.0012914 0.18738 0.0602" />
+      <parent link="${prefix}chassis_link" />
+      <child link="${prefix}l_wheel_link" />
+      <axis xyz="0 1 0" />
+      <limit effort="8.85" velocity="34.8" />
+    </joint>
+    <link name="${prefix}estop_link">
+      <inertial>
+        <origin rpy="0 0 0" xyz="0.002434512737072 -0.00330608315239905 0.00665139196650039" />
+        <mass value="0.00196130439134723" />
+        <inertia ixx="3.02810026604417E-07" ixy="-1.5862023118056E-08" ixz="3.16561396557437E-08" iyy="2.93322917127605E-07" iyz="-4.28833522751273E-08" izz="2.28513272627183E-07" />
+      </inertial>
+      <visual>
+        <origin rpy="0 0 0" xyz="0 0 0" />
+        <geometry>
+          <mesh filename="package://trina2_description/base/meshes/estop_link.STL" />
+        </geometry>
+        <material name="">
+          <color rgba="0.8 0 0 1" />
+        </material>
+      </visual>
+      <collision>
+        <origin rpy="0 0 0" xyz="0 0 0" />
+        <geometry>
+          <mesh filename="package://trina2_description/base/meshes/estop_link.STL" />
+        </geometry>
+      </collision>
+    </link>
+    <joint name="${prefix}estop_joint" type="fixed">
+      <origin rpy="1.5708 0 0" xyz="-0.12465 0.23892 0.31127" />
+      <parent link="${prefix}chassis_link" />
+      <child link="${prefix}estop_link" />
+      <axis xyz="0 0 0" />
+    </joint>
+    <link name="${prefix}laser_link">
+      <inertial>
+        <origin rpy="0 0 0" xyz="-0.0306228970175641 0.0007091682908278 0.0551974119471302" />
+        <mass value="0.00833634573995571" />
+        <inertia ixx="1.01866461240801E-06" ixy="-5.88447626567756E-08" ixz="7.83857244757914E-08" iyy="5.10039589974707E-07" iyz="-7.12664289617235E-09" izz="1.28270671527309E-06" />
+      </inertial>
+      <visual>
+        <origin rpy="0 0 0" xyz="0 0 0" />
+        <geometry>
+          <mesh filename="package://trina2_description/base/meshes/laser_link.STL" />
+        </geometry>
+        <material name="">
+          <color rgba="0.792156862745098 0.819607843137255 0.933333333333333 1" />
+        </material>
+      </visual>
+      <collision>
+        <origin rpy="0 0 0" xyz="0 0 0" />
+        <geometry>
+          <mesh filename="package://trina2_description/base/meshes/laser_link.STL" />
+        </geometry>
+      </collision>
+    </link>
+    <joint name="${prefix}laser_joint" type="fixed">
+      <origin rpy="3.14159265359 0 0" xyz="0.235 0 0.2878" />
+      <parent link="${prefix}chassis_link" />
+      <child link="${prefix}laser_link" />
+      <axis xyz="0 0 0" />
+    </joint>
+    <link name="${prefix}base_camera_link" />
+    <joint name="${prefix}base_camera_joint" type="fixed">
+      <origin rpy="0 -0.17453292519943 0" xyz="0.2645 0 0.198" />
+      <parent link="${prefix}chassis_link" />
+      <child link="${prefix}base_camera_link" />
+    </joint>
+    <link name="${prefix}base_camera_optical_frame" />
+    <joint name="${prefix}base_camera_optical_joint" type="fixed">
+      <origin rpy="1.5707963267966 0 1.5707963267966" xyz="0 0 0" />
+      <parent link="${prefix}base_camera_link" />
+      <child link="${prefix}base_camera_optical_frame" />
+    </joint>
+    <transmission name="${prefix}r_wheel_trans">
+      <type>transmission_interface/SimpleTransmission</type>
+      <joint name="${prefix}r_wheel_joint">
+          <hardwareInterface>hardware_interface/VelocityJointInterface</hardwareInterface>
+      </joint>
+      <actuator name="${prefix}r_wheel_actuator">
+          <mechanicalReduction>1</mechanicalReduction>
+      </actuator>
+    </transmission>
+    <transmission name="${prefix}l_wheel_trans">
+      <type>transmission_interface/SimpleTransmission</type>
+      <joint name="${prefix}l_wheel_joint">
+          <hardwareInterface>hardware_interface/VelocityJointInterface</hardwareInterface>
+      </joint>
+      <actuator name="${prefix}l_wheel_actuator">
+          <mechanicalReduction>1</mechanicalReduction>
+      </actuator>
+    </transmission>
+  </xacro:macro>
 </robot>

File: trina2_description/base/urdf/freight_macro.xacro (robot description, xacro)
@@ -1,9 +1,10 @@
 <?xml version="1.0"?>
 <robot name="freight" xmlns:xacro="http://www.ros.org/wiki/xacro">
-  <xacro:macro name="load_base">
+  <xacro:macro name="load_base" params="prefix">
       <!-- <xacro:include filename="$(find fetch_description)/robots/freight.urdf.xacro" /> -->
       <xacro:include filename="$(find trina2_description)/base/urdf/freight.urdf.xacro" />
+      <xacro:load_base_urdf prefix="${prefix}"/>
       <!-- Base is modeled as a big tub sitting on floor, with two wheels -->
-      <gazebo reference="chassis_link">
+      <gazebo reference="${prefix}chassis_link">
         <kp>10000000.0</kp>
         <kd>1.0</kd>
@@ -11,5 +12,5 @@
         <mu2>0.01</mu2>
       </gazebo>
-      <gazebo reference="r_wheel_link">
+      <gazebo reference="${prefix}r_wheel_link">
         <kp>10000000.0</kp>
         <kd>1.0</kd>
@@ -18,5 +19,5 @@
         <material>Gazebo/Black</material>
       </gazebo>
-      <gazebo reference="l_wheel_link">
+      <gazebo reference="${prefix}l_wheel_link">
         <kp>10000000.0</kp>
         <kd>1.0</kd>
@@ -26,18 +27,18 @@
       </gazebo>
       <!-- Color the estop -->
-      <gazebo reference="estop_link">
+      <gazebo reference="${prefix}estop_link">
         <material>Gazebo/Red</material>
       </gazebo>
-      <gazebo reference="l_wheel_joint">
+      <gazebo reference="${prefix}l_wheel_joint">
         <implicitSpringDamper>1</implicitSpringDamper>
       </gazebo>
-      <gazebo reference="r_wheel_joint">
+      <gazebo reference="${prefix}r_wheel_joint">
         <implicitSpringDamper>1</implicitSpringDamper>
       </gazebo>
-      <gazebo reference="camera_support">
+      <gazebo reference="${prefix}camera_support">
         <material>Gazebo/Black</material>
       </gazebo>
       <!-- SICK TIM561 (25m Range) -->
-      <gazebo reference="laser_link">
+      <gazebo reference="${prefix}laser_link">
       <!-- <gazebo reference="laser_link">   <! TEMPORARY FIX -->
         <sensor type="ray" name="base_laser">

File: trina2_description/base/urdf/torso.urdf.xacro (robot description, xacro)
@@ -1,10 +1,10 @@
 <?xml version="1.0"?>
 <robot name="robot_torso" xmlns:xacro="http://www.ros.org/wiki/xacro">
-    <xacro:macro name="load_torso">
+    <xacro:macro name="load_torso" params="prefix">
         <xacro:property name="mass" value="5.0" />
         <xacro:property name="width" value="0.15" />
         <xacro:property name="height" value="0.8" />
         <xacro:property name="axel_offset" value="-0.25" />
-        <link name="torso">
+        <link name="${prefix}torso">
             <collision>
                 <origin xyz="0 0 ${height/2}" rpy="0 0 0"/>
@@ -30,11 +30,11 @@
             </inertial>
         </link>
-        <joint name="torso_joint" type="fixed">
-            <parent link="chassis_link"/>
-            <child link="torso"/>
+        <joint name="${prefix}torso_joint" type="fixed">
+            <parent link="${prefix}chassis_link"/>
+            <child link="${prefix}torso"/>
             <origin xyz="-0.0 0 0.36" rpy="0 0 0"/>
             <axis xyz="0 0 1"/>
         </joint>
-        <link name="right_shoulder_link">
+        <link name="${prefix}right_shoulder_link">
             <collision>
             <origin xyz="0 0 0" rpy="0 0 0"/>
@@ -57,11 +57,11 @@
             </inertial>
         </link>
-        <joint name="right_shoulder_to_torso_joint" type="fixed">
-            <child link="right_shoulder_link" />
-            <parent link="torso" />
+        <joint name="${prefix}right_shoulder_to_torso_joint" type="fixed">
+            <child link="${prefix}right_shoulder_link" />
+            <parent link="${prefix}torso" />
             <origin xyz="0 0 0.7" rpy="1.57 0 0" />
             <axis xyz="0 0 1"/>
         </joint>
-        <link name="left_shoulder_link">
+        <link name="${prefix}left_shoulder_link">
             <collision>
             <origin xyz="0 0 0" rpy="0 0 0"/>
@@ -84,7 +84,7 @@
             </inertial>
         </link>
-        <joint name="left_shoulder_to_torso_joint" type="fixed">
-            <child link="left_shoulder_link" />
-            <parent link="torso" />
+        <joint name="${prefix}left_shoulder_to_torso_joint" type="fixed">
+            <child link="${prefix}left_shoulder_link" />
+            <parent link="${prefix}torso" />
             <origin xyz="0 0 0.7" rpy="-1.57 0 0" />
             <axis xyz="0 0 1"/>

File: trina2_description/camera/urdf/_d435.gazebo.xacro (robot description, xacro)
@@ -6,5 +6,5 @@
 <robot xmlns:xacro="http://ros.org/wiki/xacro">
   <xacro:macro name="gazebo_d435" params="camera_name reference_link
-                                          topics_ns color_optical_frame
+                                          color_optical_frame
                                           fov:=69.4 width:=1920 height:=1080
                                           update_rate:=30" >
