Commit message: add tf_prefix to urdf

File: trina2_description/camera/urdf/_d435.urdf.xacro (robot description, xacro)
@@ -9,5 +9,5 @@
   <!--File includes-->
   <xacro:include filename="$(find trina2_description)/camera/urdf/_d435.gazebo.xacro"/>
-  <xacro:macro name="sensor_d435" params="name:=camera topics_ns:=camera parent
+  <xacro:macro name="sensor_d435" params="name:=camera prefix:=camera/ parent
                                           fov:=69.4 width:=1920 height:=1080
                                           update_rate:=60 wide_flag:=false *origin">
@@ -30,20 +30,20 @@
     <xacro:property name="d435_cam_depth_py" value="0.0175"/>
     <xacro:property name="d435_cam_depth_pz" value="${d435_cam_height/2}"/>
-    <material name="${name}_aluminum">
+    <material name="${prefix}aluminum">
 	  <color rgba="0.5 0.5 0.5 1"/>
     </material>
     <!-- camera body, with origin at bottom screw mount -->
-    <joint name="${name}_joint" type="fixed">
+    <joint name="${prefix}joint" type="fixed">
       <xacro:insert_block name="origin" />
       <parent link="${parent}"/>
-      <child link="${name}_bottom_screw_frame" />
+      <child link="${prefix}bottom_screw_frame" />
     </joint>
-    <link name="${name}_bottom_screw_frame"/>
-    <joint name="${name}_link_joint" type="fixed">
+    <link name="${prefix}bottom_screw_frame"/>
+    <joint name="${prefix}link_joint" type="fixed">
       <origin xyz="0 ${d435_cam_depth_py} ${d435_cam_depth_pz}" rpy="0 0 0"/>
-      <parent link="${name}_bottom_screw_frame"/>
-      <child link="${name}_link" />
+      <parent link="${prefix}bottom_screw_frame"/>
+      <child link="${prefix}link" />
     </joint>
-    <link name="${name}_link">
+    <link name="${prefix}link">
       <visual>
       <origin xyz="${d435_cam_mount_from_center_offset} ${-d435_cam_depth_py} 0" rpy="${M_PI/2} 0 ${M_PI/2}"/>
@@ -53,5 +53,5 @@
           <!--<mesh filename="package://realsense2_description/meshes/d435/d435.dae" />-->
         </geometry>
-        <material name="${name}_aluminum"/>
+        <material name="${prefix}aluminum"/>
       </visual>
       <collision>
@@ -71,59 +71,58 @@
     </link>
     <!-- camera depth joints and links -->
-    <joint name="${name}_depth_joint" type="fixed">
+    <joint name="${prefix}depth_joint" type="fixed">
       <origin xyz="0 0 0" rpy="0 0 0"/>
-      <parent link="${name}_link"/>
-      <child link="${name}_depth_frame" />
+      <parent link="${prefix}link"/>
+      <child link="${prefix}depth_frame" />
     </joint>
-    <link name="${name}_depth_frame"/>
-    <joint name="${name}_depth_optical_joint" type="fixed">
+    <link name="${prefix}depth_frame"/>
+    <joint name="${prefix}depth_optical_joint" type="fixed">
       <origin xyz="0 0 0" rpy="${-M_PI/2} 0 ${-M_PI/2}" />
-      <parent link="${name}_depth_frame" />
-      <child link="${name}_depth_optical_frame" />
+      <parent link="${prefix}depth_frame" />
+      <child link="${prefix}depth_optical_frame" />
     </joint>
-    <link name="${name}_depth_optical_frame"/>
+    <link name="${prefix}depth_optical_frame"/>
     <!-- camera left IR joints and links -->
-    <joint name="${name}_left_ir_joint" type="fixed">
+    <joint name="${prefix}left_ir_joint" type="fixed">
       <origin xyz="0 ${d435_cam_depth_to_left_ir_offset} 0" rpy="0 0 0" />
-      <parent link="${name}_depth_frame" />
-      <child link="${name}_left_ir_frame" />
+      <parent link="${prefix}depth_frame" />
+      <child link="${prefix}left_ir_frame" />
     </joint>
-    <link name="${name}_left_ir_frame"/>
-    <joint name="${name}_left_ir_optical_joint" type="fixed">
+    <link name="${prefix}left_ir_frame"/>
+    <joint name="${prefix}left_ir_optical_joint" type="fixed">
       <origin xyz="0 0 0" rpy="${-M_PI/2} 0 ${-M_PI/2}" />
-      <parent link="${name}_left_ir_frame" />
-      <child link="${name}_left_ir_optical_frame" />
+      <parent link="${prefix}left_ir_frame" />
+      <child link="${prefix}left_ir_optical_frame" />
     </joint>
-    <link name="${name}_left_ir_optical_frame"/>
+    <link name="${prefix}left_ir_optical_frame"/>
     <!-- camera right IR joints and links -->
-    <joint name="${name}_right_ir_joint" type="fixed">
+    <joint name="${prefix}right_ir_joint" type="fixed">
       <origin xyz="0 ${d435_cam_depth_to_right_ir_offset} 0" rpy="0 0 0" />
-      <parent link="${name}_depth_frame" />
-      <child link="${name}_right_ir_frame" />
+      <parent link="${prefix}depth_frame" />
+      <child link="${prefix}right_ir_frame" />
     </joint>
-    <link name="${name}_right_ir_frame"/>
-    <joint name="${name}_right_ir_optical_joint" type="fixed">
+    <link name="${prefix}right_ir_frame"/>
+    <joint name="${prefix}right_ir_optical_joint" type="fixed">
       <origin xyz="0 0 0" rpy="${-M_PI/2} 0 ${-M_PI/2}" />
-      <parent link="${name}_right_ir_frame" />
-      <child link="${name}_right_ir_optical_frame" />
+      <parent link="${prefix}right_ir_frame" />
+      <child link="${prefix}right_ir_optical_frame" />
     </joint>
-    <link name="${name}_right_ir_optical_frame"/>
+    <link name="${prefix}right_ir_optical_frame"/>
     <!-- camera color joints and links -->
-    <joint name="${name}_color_joint" type="fixed">
+    <joint name="${prefix}color_joint" type="fixed">
       <origin xyz="0 ${d435_cam_depth_to_color_offset} 0" rpy="0 0 0" />
-      <parent link="${name}_depth_frame" />
-      <child link="${name}_color_frame" />
+      <parent link="${prefix}depth_frame" />
+      <child link="${prefix}color_frame" />
     </joint>
-    <link name="${name}_color_frame"/>
-    <joint name="${name}_color_optical_joint" type="fixed">
+    <link name="${prefix}color_frame"/>
+    <joint name="${prefix}color_optical_joint" type="fixed">
       <origin xyz="0 0 0" rpy="${-M_PI/2} 0 ${-M_PI/2}" />
-      <parent link="${name}_color_frame" />
-      <child link="${name}_color_optical_frame" />
+      <parent link="${prefix}color_frame" />
+      <child link="${prefix}color_optical_frame" />
     </joint>
-    <link name="${name}_color_optical_frame"/>
+    <link name="${prefix}color_optical_frame"/>
     <!-- Realsense Gazebo Plugin -->
     <!-- Normal camera -->
-    <xacro:gazebo_d435 camera_name="${name}" reference_link="${name}_link"
-                      topics_ns="${topics_ns}"
+    <xacro:gazebo_d435 camera_name="${name}" reference_link="${prefix}link"
                       color_optical_frame="${name}_color_optical_frame"
                       fov="${fov}" width="${width}" height="${height}"
@@ -131,6 +130,5 @@
     <!-- Wide camera -->
     <xacro:if value="${wide_flag}">
-    <xacro:gazebo_d435 camera_name="${name}_wide" reference_link="${name}_link"
-                      topics_ns="${topics_ns}_wide"
+    <xacro:gazebo_d435 camera_name="${name}_wide" reference_link="${prefix}link"
                       color_optical_frame="${name}_color_optical_frame"
                       fov="114" width="${1.3125*width}" height="${height}"

File: trina2_description/camera/urdf/arm_camera.urdf.xacro (robot description, xacro)
@@ -1,8 +1,8 @@
 <?xml version="1.0"?>
 <robot name="main_camera" xmlns:xacro="http://www.ros.org/wiki/xacro">
-    <xacro:macro name="load_arm_camera" params="prefix arm_camera_base
+    <xacro:macro name="load_arm_camera" params="prefix camera_name arm_camera_base
                                                 fov:=69.4 width:=1920 height:=1080
                                                 update_rate:=60 wide_flag:=true">
-        <link name="${prefix}camera_support">
+        <link name="${prefix}support">
             <collision>
             <origin xyz="0 0 0" rpy="0 0 0"/>
@@ -25,12 +25,13 @@
             </inertial>
         </link>
-        <joint name="${prefix}camera_support_joint" type="fixed">
+        <joint name="${prefix}support_joint" type="fixed">
             <parent link="${arm_camera_base}"/>
-            <child link="${prefix}camera_support"/>
+            <child link="${prefix}support"/>
             <origin xyz="0 0 0" rpy="0 -1.57 1.57"/>
             <axis xyz="0 0 1"/>
         </joint>
         <xacro:include filename="$(find trina2_description)/camera/urdf/_d435.urdf.xacro"/>
-        <xacro:sensor_d435 name="${prefix}cam" parent="${prefix}camera_support"
+        <xacro:sensor_d435 name="${camera_name}" prefix="${prefix}"
+                           parent="${prefix}support"
                            fov="${fov}" width="${width}" height="${height}"
                            update_rate="${update_rate}" wide_flag="${wide_flag}">

File: trina2_description/camera/urdf/main_camera_support.urdf.xacro (robot description, xacro)
@@ -1,5 +1,5 @@
 <?xml version="1.0"?>
 <robot name="main_camera" xmlns:xacro="http://www.ros.org/wiki/xacro">
-    <xacro:macro name="load_main_camera" params="prefix main_camera_base
+    <xacro:macro name="load_main_camera" params="prefix camera_name main_camera_base
                                                  fov:=69.4 width:=1920 height:=1080
                                                  update_rate:=60 wide_flag:=true">
@@ -8,5 +8,5 @@
         <xacro:property name="height_support" value="0.02" />
         <xacro:property name="axel_offset" value="-0.25" />
-        <link name="${prefix}camera_support">
+        <link name="${prefix}support">
             <collision>
             <origin xyz="0 0 ${height_support/2}" rpy="0 0 0"/>
@@ -32,11 +32,11 @@
             </inertial>
         </link>
-        <joint name="${prefix}camera_support_joint" type="fixed">
+        <joint name="${prefix}support_joint" type="fixed">
             <parent link="${main_camera_base}"/>
-            <child link="${prefix}camera_support"/>
+            <child link="${prefix}support"/>
             <origin xyz="${0.075-width_support/2} 0 0.8" rpy="0 0 0"/>
             <axis xyz="0 0 1"/>
         </joint>
-        <link name="${prefix}camera_yaw_link">
+        <link name="${prefix}yaw_link">
             <collision>
             <origin xyz="0 0 0.02" rpy="0 0 0"/>
@@ -62,12 +62,12 @@
             </inertial>
         </link>
-        <joint name="${prefix}camera_yaw_joint" type="revolute">
-            <parent link="${prefix}camera_support"/>
-            <child link="${prefix}camera_yaw_link"/>
+        <joint name="${prefix}yaw_joint" type="revolute">
+            <parent link="${prefix}support"/>
+            <child link="${prefix}yaw_link"/>
             <origin xyz="0 0 ${height_support}" rpy="0 0 0"/>
             <axis xyz="0 0 1"/>
             <limit lower="-1.047" upper="1.047" effort="20" velocity="1.0" />
         </joint>
-        <link name="${prefix}camera_pitch_link">
+        <link name="${prefix}pitch_link">
             <collision>
             <origin xyz="0 0 0" rpy="0 0 0"/>
@@ -93,31 +93,32 @@
             </inertial>
         </link>
-        <joint name="${prefix}camera_pitch_joint" type="revolute">
-            <parent link="${prefix}camera_yaw_link"/>
-            <child link="${prefix}camera_pitch_link"/>
+        <joint name="${prefix}pitch_joint" type="revolute">
+            <parent link="${prefix}yaw_link"/>
+            <child link="${prefix}pitch_link"/>
             <origin xyz="0.02 0 0.02" rpy="1.57 0 0"/>
             <axis xyz="0 0 1"/>
             <limit lower="-1.047" upper="1.047" effort="20" velocity="1.0" />
         </joint>
-        <transmission name="${prefix}camera_yaw_trans">
+        <transmission name="${prefix}yaw_trans">
             <type>transmission_interface/SimpleTransmission</type>
-            <joint name="${prefix}camera_yaw_joint">
+            <joint name="${prefix}yaw_joint">
                 <hardwareInterface>hardware_interface/EffortJointInterface</hardwareInterface>
             </joint>
-            <actuator name="${prefix}camera_yaw_actuator">
+            <actuator name="${prefix}yaw_actuator">
                 <mechanicalReduction>1</mechanicalReduction>
             </actuator>
         </transmission>
-        <transmission name="${prefix}camera_pitch_trans">
+        <transmission name="${prefix}pitch_trans">
             <type>transmission_interface/SimpleTransmission</type>
-            <joint name="${prefix}camera_pitch_joint">
+            <joint name="${prefix}pitch_joint">
                 <hardwareInterface>hardware_interface/EffortJointInterface</hardwareInterface>
             </joint>
-            <actuator name="${prefix}camera_pitch_actuator">
+            <actuator name="${prefix}pitch_actuator">
                 <mechanicalReduction>1</mechanicalReduction>
             </actuator>
         </transmission>
         <xacro:include filename="$(find trina2_description)/camera/urdf/_d435.urdf.xacro"/>
-        <xacro:sensor_d435 name="${prefix}cam" parent="${prefix}camera_pitch_link"
+        <xacro:sensor_d435 name="${camera_name}" prefix="${prefix}"
+                           parent="${prefix}pitch_link"
                            fov="${fov}" width="${width}" height="${height}"
                            update_rate="${update_rate}"  wide_flag="${wide_flag}">

File: trina2_description/robots/urdf/trina2.xacro (robot description, xacro)
@@ -7,6 +7,8 @@
     <xacro:arg name="gripper" default="robotiq_2f_85" />
     <xacro:arg name="sim" default="true" />
-    <xacro:arg name="right_prefix" default="right_arm_" />
-    <xacro:arg name="left_prefix" default="left_arm_" />
+    <xacro:arg name="robot_name" default="trina2" />
+    <xacro:arg name="prefix" default="$(arg robot_name)/" />
+    <xacro:arg name="right_prefix" default="$(arg prefix)right_arm_" />
+    <xacro:arg name="left_prefix" default="$(arg prefix)left_arm_" />
     <!-- Include files -->
     <xacro:include filename="$(find trina2_description)/base/urdf/freight_macro.xacro" />
@@ -16,23 +18,23 @@
     <xacro:include filename="$(find trina2_description)/camera/urdf/arm_camera.urdf.xacro" />
     <!-- Load the base -->
-    <xacro:load_base/>
+    <xacro:load_base prefix="$(arg prefix)"/>
     <!-- Load torso -->
-    <xacro:load_torso/>
+    <xacro:load_torso prefix="$(arg prefix)"/>
     <!-- Load the right arm -->
     <xacro:load_robot arm="$(arg arm)" gripper="$(arg gripper)" dof="$(arg dof)"
                     vision="$(arg vision)" sim="$(arg sim)"
-                    prefix="$(arg right_prefix)" parent="right_shoulder_link"/>
+                    prefix="$(arg right_prefix)" parent="$(arg prefix)right_shoulder_link"/>
     <!-- Load arm camera -->
-    <xacro:load_arm_camera prefix="$(arg right_prefix)" arm_camera_base="$(arg right_prefix)camera_link"
+    <xacro:load_arm_camera prefix="$(arg right_prefix)cam_" camera_name="right_arm_cam" arm_camera_base="$(arg right_prefix)camera_link"
                            width="858" height="720" update_rate="30" wide_flag="true"/>
     <!-- Load the left arm -->
     <xacro:load_robot arm="$(arg arm)" gripper="$(arg gripper)" dof="$(arg dof)"
                     vision="$(arg vision)" sim="$(arg sim)"
-                    prefix="$(arg left_prefix)" parent="left_shoulder_link"/>
+                    prefix="$(arg left_prefix)" parent="$(arg prefix)left_shoulder_link"/>
     <!-- Load arm camera -->
-    <xacro:load_arm_camera prefix="$(arg left_prefix)" arm_camera_base="$(arg left_prefix)camera_link"
+    <xacro:load_arm_camera prefix="$(arg left_prefix)cam_" camera_name="left_arm_cam" arm_camera_base="$(arg left_prefix)camera_link"
                            width="858" height="720" update_rate="30" wide_flag="true"/>
     <!-- Load main camera -->
-    <xacro:load_main_camera prefix="main_" main_camera_base="torso"
+    <xacro:load_main_camera prefix="$(arg prefix)main_cam_" camera_name="main_cam" main_camera_base="$(arg prefix)torso"
                             width="858" height="720" update_rate="30" wide_flag="true"/>
     <!-- Load gazebo control pulgin ONLY ONCE -->
